File: RubyPad.sch (KiCad schematic (older format))
At the start: 24 parts, among them J1 USB_mini_micro_B, K1 KEYSW, K2 KEYSW, K3 KEYSW, K4 KEYSW, SW1 SW_PUSH, U1 ATMEGA32U4, X1 XTAL_GND

Commit message: Redone the pcb again but forgot the 'fill area' thing
Parts:
- added D3, D6: D, keyboard_parts:D_SOD123_axial, symbol RubyPad-rescue:D-TMK_parts
- added K3, K6: KEYSW, HotSwap:Kailh_MX_Socket, symbol RubyPad-rescue:KEYSW-TMK_parts
- C1: renamed from C8; footprint Capacitor_SMD:C_0805_2012Metric_Pad1.15x1.40mm_HandSolder -> Capacitor_SMD:C_0805_2012Metric_Pad1.18x1.45mm_HandSolder; symbol TMK_parts:C -> RubyPad-rescue:C-TMK_parts
- C2: renamed from C1; footprint Capacitor_SMD:C_0805_2012Metric_Pad1.15x1.40mm_HandSolder -> Capacitor_SMD:C_0805_2012Metric_Pad1.18x1.45mm_HandSolder
- C3: renamed from C2; footprint Capacitor_SMD:C_0805_2012Metric_Pad1.15x1.40mm_HandSolder -> Capacitor_SMD:C_0805_2012Metric_Pad1.18x1.45mm_HandSolder
- C4: renamed from C3; footprint Capacitor_SMD:C_0805_2012Metric_Pad1.15x1.40mm_HandSolder -> Capacitor_SMD:C_0805_2012Metric_Pad1.18x1.45mm_HandSolder
- C5: renamed from C4; footprint Capacitor_SMD:C_0805_2012Metric_Pad1.15x1.40mm_HandSolder -> Capacitor_SMD:C_0805_2012Metric_Pad1.18x1.45mm_HandSolder
- C6: renamed from C5; footprint Capacitor_SMD:C_0805_2012Metric_Pad1.15x1.40mm_HandSolder -> Capacitor_SMD:C_0805_2012Metric_Pad1.18x1.45mm_HandSolder
- C7: renamed from C6; footprint Capacitor_SMD:C_0805_2012Metric_Pad1.15x1.40mm_HandSolder -> Capacitor_SMD:C_0805_2012Metric_Pad1.18x1.45mm_HandSolder
- C8: renamed from C7; footprint Capacitor_SMD:C_0805_2012Metric_Pad1.15x1.40mm_HandSolder -> Capacitor_SMD:C_0805_2012Metric_Pad1.18x1.45mm_HandSolder
- D1: symbol TMK_parts:D -> RubyPad-rescue:D-TMK_parts
- D2: renamed from D3; symbol TMK_parts:D -> RubyPad-rescue:D-TMK_parts
- D4: renamed from D2; symbol TMK_parts:D -> RubyPad-rescue:D-TMK_parts
- D5: renamed from D4; symbol TMK_parts:D -> RubyPad-rescue:D-TMK_parts
- J1: symbol TMK_parts:USB_mini_micro_B -> RubyPad-rescue:USB_mini_micro_B-TMK_parts
- K1: footprint keebs:Mx_Alps_100 -> HotSwap:Kailh_MX_Socket; symbol TMK_parts:KEYSW -> RubyPad-rescue:KEYSW-TMK_parts
- K2: renamed from K3; footprint keebs:Mx_Alps_100 -> HotSwap:Kailh_MX_Socket; symbol TMK_parts:KEYSW -> RubyPad-rescue:KEYSW-TMK_parts
- K4: renamed from K2; footprint keebs:Mx_Alps_100 -> HotSwap:Kailh_MX_Socket; symbol TMK_parts:KEYSW -> RubyPad-rescue:KEYSW-TMK_parts
- K5: renamed from K4; footprint keebs:Mx_Alps_100 -> HotSwap:Kailh_MX_Socket; symbol TMK_parts:KEYSW -> RubyPad-rescue:KEYSW-TMK_parts
- R1: renamed from R2; footprint Resistor_SMD:R_0805_2012Metric_Pad1.15x1.40mm_HandSolder -> Resistor_SMD:R_0805_2012Metric_Pad1.20x1.40mm_HandSolder; symbol TMK_parts:R -> RubyPad-rescue:R-TMK_parts
- R2: renamed from R3; footprint Resistor_SMD:R_0805_2012Metric_Pad1.15x1.40mm_HandSolder -> Resistor_SMD:R_0805_2012Metric_Pad1.20x1.40mm_HandSolder; symbol TMK_parts:R -> RubyPad-rescue:R-TMK_parts
- R3: renamed from R1; footprint Resistor_SMD:R_0805_2012Metric_Pad1.15x1.40mm_HandSolder -> Resistor_SMD:R_0805_2012Metric_Pad1.20x1.40mm_HandSolder; symbol TMK_parts:R -> RubyPad-rescue:R-TMK_parts
- R4: footprint Resistor_SMD:R_0805_2012Metric_Pad1.15x1.40mm_HandSolder -> Resistor_SMD:R_0805_2012Metric_Pad1.20x1.40mm_HandSolder; symbol TMK_parts:R -> RubyPad-rescue:R-TMK_parts
- SW1: footprint Button_Switch_SMD:SW_SPST_TL3342 -> Keebio-Parts:SW_SPST_3x3; symbol TMK_parts:SW_PUSH -> RubyPad-rescue:SW_PUSH-TMK_parts
- U1: symbol TMK_parts:ATMEGA32U4 -> RubyPad-rescue:ATMEGA32U4-TMK_parts
- X1: symbol TMK_parts:XTAL_GND -> RubyPad-rescue:XTAL_GND-TMK_parts
Connections:
- net row0: now also D3.1
- net row1: now also D6.1
- net col2: now reaches U1.37 (PF6)
- net col2: now also K3.1, K6.1
- new net: D3.2, K3.2
- new net: D6.2, K6.2
- no-connect marks 24 -> 23
Other:
- moved on the sheet: D1, D2, D4, D5, K1, K2, K4, K5
