File: rubypad.kicad_pcb (KiCad board)
At the start: 2 copper layers, 32 parts, among them J1 HRO-TYPE-C, SW1 SW_Push, SW2 RotaryEncoder_Switch, U1 ATmega32U4-A, Y1 16MHz

Commit message: resuming works
Parts:
- moved MX3 77.2 mm to (39.6, 65.5)
- moved MX2 77.1 mm to (59.9, 65.5)
- moved MX6 71.5 mm to (39.6, 85.9)
- moved SW1 70.4 mm to (112.8, 136.7)
- moved MX5 51.2 mm to (59.9, 85.9)
- moved Y1 50.5 mm to (133.6, 89.4)
- moved D1 39.4 mm to (43.9, 120.1)
- moved D4 39.4 mm to (43.9, 116.9)
- moved D7 39.4 mm to (43.9, 123.2)
- moved C1 39.4 mm to (69.3, 119.9)
- moved C2 39.4 mm to (67.4, 122.9)
- moved C3 39.4 mm to (57.8, 122.9)
- moved C4 39.4 mm to (64.5, 119.9)
- moved C5 39.4 mm to (62.6, 122.9)
- moved C6 39.4 mm to (69.3, 116.9)
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