File: rubypad.kicad_pcb (KiCad board)
At the start: 2 copper layers, 32 parts, among them J1 HRO-TYPE-C, SW1 SW_Push, SW2 RotaryEncoder_Switch, U1 ATmega32U4-A, Y1 16MHz

Commit message: update
Parts:
- C1, C2, C3, C5, C6, C7, C8, R6, U1, Y1: moved to B.Cu
- moved SW1 102.2 mm to (97.5, 35.6), turned to -90 degrees
- moved C8 93.4 mm to (48.7, 49.3)
- moved R5 88.7 mm to (43.7, 45.3), turned to -90 degrees
- moved C7 87.5 mm to (56.4, 51.4), turned to -90 degrees
- moved Y1 83.8 mm to (56.4, 56.9), turned to 135 degrees
- moved C5 81.9 mm to (37.6, 52.4), turned to -90 degrees
- moved R3 79.9 mm to (49.3, 43.2), turned to 180 degrees
- moved R4 78.5 mm to (45.8, 45.3), turned to -90 degrees
- moved C2 77.3 mm to (41.1, 49.3), turned to 180 degrees
- moved C6 74.9 mm to (56.4, 62.6), turned to 90 degrees
- moved C4 72.5 mm to (53.4, 53.0), turned to 90 degrees
- moved C1 66.9 mm to (37.6, 61.6), turned to -90 degrees
- moved C3 62.6 mm to (49.8, 64.7)
- moved SW2 50.9 mm to (67.6, 46.2), turned to 90 degrees
- moved D1 46.2 mm to (67.6, 36.1), turned to 180 degrees
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Connections:
- U1 pad 29: unconnected-(U1-Pad29) -> col0
- U1 pad 30: unconnected-(U1-Pad30) -> col1
- U1 pad 31: unconnected-(U1-Pad31) -> col2

Commit message: add to schematic
Parts:
- moved R1 8.87 mm to (89.4, 43.2)
- moved SW1 8.87 mm to (89.4, 39.1)
Other:
- board outline added: 65 x 77.5 mm
Changed lines of the file:
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@@
   )
   (footprint "reversible-kicad-footprints:PushButton_4.5mm" (layer "F.Cu")
-    (at 97.536 35.56 -90)
+    (at 89.408 39.116 -90)
     (property "Sheetfile" "rubypad.kicad_sch")
     (property "Sheetname" "")
@@
   )
   (footprint "Resistor_SMD:R_0805_2012Metric_Pad1.20x1.40mm_HandSolder" (layer "F.Cu")
-    (at 97.552 39.624)
+    (at 89.424 43.18)
     (descr "Resistor SMD 0805 (2012 Metric), square (rectangular) end terminal, IPC_7351 nominal with elongated pad for handsoldering. (Body size source: IPC-SM-782 page 72, https://www.pcb-3d.com/wordpress/wp-content/uploads/ipc-sm-782a_amendment_1_and_2.pdf), generated with kicad-footprint-generator")
     (tags "resistor handsolder")
@@
     )
   )
+  (gr_line (start 100 107.5) (end 100 35) (layer "Edge.Cuts") (width 0.1))
+  (gr_line (start 97.5 32.5) (end 37.5 32.5) (layer "Edge.Cuts") (width 0.1))
+  (gr_arc (start 97.5 32.5) (mid 99.267767 33.232233) (end 100 35) (layer "Edge.Cuts") (width 0.1))
+  (gr_arc (start 37.5 110) (mid 35.732233 109.267767) (end 35 107.5) (layer "Edge.Cuts") (width 0.1))
+  (gr_line (start 35 35) (end 35 107.5) (layer "Edge.Cuts") (width 0.1))
+  (gr_arc (start 100 107.5) (mid 99.267767 109.267767) (end 97.5 110) (layer "Edge.Cuts") (width 0.1))
+  (gr_line (start 37.5 110) (end 97.5 110) (layer "Edge.Cuts") (width 0.1))
+  (gr_arc (start 35 35) (mid 35.732233 33.232233) (end 37.5 32.5) (layer "Edge.Cuts") (width 0.1))
 )

Commit message: changes and complete
Parts:
- C3, R6: moved to F.Cu
- moved D1 24.9 mm to (68.0, 61.0), turned to 0 degrees
- moved R1 11.6 mm to (94.5, 53.6)
- moved SW1 11.6 mm to (94.5, 49.5)
- moved SW2 3.27 mm to (67.5, 49.5), turned to -90 degrees
- moved C4 3.23 mm to (52.0, 50.0)
- moved D5 2.72 mm to (87.9, 100.9)
- moved D6 2.72 mm to (67.6, 100.9)
- moved D7 2.72 mm to (47.2, 100.9)
- moved MX4 2.72 mm to (87.9, 94.8)
- moved MX5 2.72 mm to (67.6, 94.8)
- moved MX6 2.72 mm to (47.2, 94.8)
- moved D2 2.72 mm to (87.9, 80.6)
- moved D3 2.72 mm to (68.1, 80.6)
- moved D4 2.72 mm to (47.2, 80.6)
- moved MX1 2.72 mm to (87.9, 74.5)
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Connections:
- U1 pad 20: unconnected-(U1-Pad20) -> col0
- U1 pad 21: unconnected-(U1-Pad21) -> col1
- U1 pad 22: unconnected-(U1-Pad22) -> col2
- U1 pad 28: unconnected-(U1-Pad28) -> row0
- U1 pad 29: col0 -> row1
- U1 pad 30: col1 -> row2
- U1 pad 31: col2 -> unconnected-(U1-Pad31)
- U1 pad 38: unconnected-(U1-Pad38) -> encA
- U1 pad 39: unconnected-(U1-Pad39) -> encC
- U1 pad 40: unconnected-(U1-Pad40) -> encB
Routing:
- net VCC: track 0.00 -> 100.8 mm, vias 0 -> 3
- net row2: track 0.00 -> 84.0 mm, vias 0 -> 1
- net row1: track 0.00 -> 63.7 mm, vias 0 -> 1
- net col0: track 0.00 -> 56.3 mm, vias 0 -> 2
- net col1: track 0.00 -> 54.0 mm
- net encC: track 0.00 -> 52.1 mm, vias 0 -> 1
- net Net-(R1-Pad2): track 0.00 -> 51.5 mm
- net encB: track 0.00 -> 46.8 mm, vias 0 -> 1
- net col2: track 0.00 -> 41.5 mm
- net row0: track 0.00 -> 26.2 mm, vias 0 -> 1
- net GND: track 0.00 -> 18.8 mm
- net Net-(D6-Pad2): track 0.00 -> 13.2 mm
- net Net-(D7-Pad2): track 0.00 -> 13.2 mm
- net Net-(D5-Pad2): track 0.00 -> 13.2 mm
- net Net-(D4-Pad2): track 0.00 -> 13.2 mm
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- added copper zone on B.Cu, net GND
- added copper zone on F.Cu, net GND
Other:
- board size 65 x 77.5 mm -> 65 x 72 mm

Commit message: udpate - going to redo pcb again
Parts:
- added G***: LOGO, rubypad-footprints:logo, F.Cu at (78.7, 41.1)
- added G***: LOGO, rubypad-footprints:logo, B.Cu at (92.7, 41.1)
- moved R1 11.4 mm to (94.0, 42.2)
- moved SW1 10.4 mm to (94.0, 39.1)
- moved D1 2.43 mm to (67.3, 58.7)
- moved C6 1.89 mm to (57.7, 61.2), turned to 180 degrees
- moved C7 1.15 mm to (57.2, 52.3), turned to 180 degrees
Routing:
- net encA: track 0.00 -> 56.7 mm, vias 0 -> 1
- net col0: track 56.3 -> 68.7 mm, vias 2 -> 0
- net D-: track 12.2 -> 4.25 mm
- net GND: track 18.8 -> 24.9 mm, vias 0 -> 1
- net Net-(R1-Pad2): track 51.5 -> 57.0 mm
- net Net-(C6-Pad2): track 9.25 -> 6.31 mm
- net Net-(D1-Pad2): track 4.52 -> 2.44 mm
- net row0: track 26.2 -> 28.2 mm
- net Net-(D3-Pad2): track 13.1 -> 14.1 mm, vias 2 -> 0
- net VCC: track 100.8 -> 100.0 mm

Commit message: udpate
Parts:
- removed G*** (x2): LOGO, rubypad-footprints:logo
- C1, C2, C5, C6, C7, C8, U1: moved to F.Cu
- J1: moved to B.Cu
- Y1: footprint Crystal:Crystal_SMD_3225-4Pin_3.2x2.5mm_HandSoldering -> Crystal:Crystal_SMD_SeikoEpson_TSX3225-4Pin_3.2x2.5mm_HandSoldering; moved to F.Cu
- moved R2 229.6 mm to (247.4, 142.7)
- moved R6 225.8 mm to (252.1, 142.7), turned to 0 degrees
- moved R5 225.3 mm to (240.0, 156.0), turned to 0 degrees
- moved R3 223.2 mm to (247.4, 145.7), turned to 0 degrees
- moved R4 219.9 mm to (253.9, 114.9), turned to 0 degrees
- moved C2 202.4 mm to (213.1, 151.4), turned to 0 degrees
- moved C8 196.5 mm to (213.1, 156.5)
- moved C1 193.9 mm to (205.8, 158.2), turned to 0 degrees
- moved C5 193.7 mm to (206.7, 147.0), turned to 0 degrees
- moved R1 186.7 mm to (247.4, 148.6)
- moved C4 186.3 mm to (207.5, 152.7), turned to 0 degrees
- moved C3 178.3 mm to (202.7, 156.5)
- moved D4 153.2 mm to (188.0, 141.1)
- moved D7 148.2 mm to (188.0, 147.4)
- moved D3 144.2 mm to (208.1, 115.0)
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Connections:
- U1 pad 20: col0 -> unconnected-(U1-Pad20)
- U1 pad 21: col1 -> unconnected-(U1-Pad21)
- U1 pad 22: col2 -> unconnected-(U1-Pad22)
- U1 pad 28: row0 -> unconnected-(U1-Pad28)
- U1 pad 29: row1 -> unconnected-(U1-Pad29)
- U1 pad 30: row2 -> unconnected-(U1-Pad30)
- U1 pad 38: encA -> unconnected-(U1-Pad38)
- U1 pad 39: encC -> unconnected-(U1-Pad39)
- U1 pad 40: encB -> unconnected-(U1-Pad40)
Routing:
- net VCC: track 100.0 -> 0.00 mm, vias 3 -> 0
- net row2: track 84.0 -> 0.00 mm, vias 1 -> 0
- net col0: track 68.7 -> 0.00 mm
- net row1: track 63.7 -> 0.00 mm, vias 1 -> 0
- net Net-(R1-Pad2): track 57.0 -> 0.00 mm
- net encA: track 56.7 -> 0.00 mm, vias 1 -> 0
- net col1: track 54.0 -> 0.00 mm
- net encC: track 52.1 -> 0.00 mm, vias 1 -> 0
- net encB: track 46.8 -> 0.00 mm, vias 1 -> 0
- net col2: track 41.5 -> 0.00 mm
- net row0: track 28.2 -> 0.00 mm, vias 1 -> 0
- net GND: track 24.9 -> 0.00 mm, vias 1 -> 0
- net Net-(D3-Pad2): track 14.1 -> 0.00 mm
- net Net-(D6-Pad2): track 13.2 -> 0.00 mm
- net Net-(D7-Pad2): track 13.2 -> 0.00 mm
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- removed copper zone on B.Cu, net GND
- removed copper zone on F.Cu, net GND
Other:
- board outline removed

Commit message: updates
Parts:
- added F1: 500mA, Fuse:Fuse_1206_3216Metric_Pad1.42x1.75mm_HandSolder, F.Cu at (81.3, 85.1)
- C2, C6, C7, C8, R2, R3, R6, U1, Y1: moved to B.Cu
- moved R2 177.3 mm to (81.5, 80.0)
- moved R3 174.2 mm to (86.1, 80.0), turned to 180 degrees
- moved R4 169.9 mm to (85.1, 96.2), turned to -90 degrees
- moved R5 168.4 mm to (82.5, 96.2), turned to -90 degrees
- moved R1 137.3 mm to (128.5, 80.0), turned to 180 degrees
- moved R6 129.2 mm to (137.2, 83.8)
- moved C1 105.8 mm to (130.6, 83.8)
- moved C2 104.4 mm to (124.5, 96.3), turned to -90 degrees
- moved C8 101.0 mm to (128.3, 101.6), turned to 180 degrees
- moved D4 95.3 mm to (96.5, 114.3), turned to 90 degrees
- moved C3 94.1 mm to (139.7, 86.6), turned to 90 degrees
- moved D7 92.6 mm to (96.5, 133.3), turned to 90 degrees
- moved D3 92.5 mm to (115.6, 114.3), turned to 90 degrees
- moved C4 88.2 mm to (139.7, 96.3), turned to -90 degrees
- moved C5 84.7 mm to (136.9, 99.1)
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Connections:
- net Net-(C6-Pad2) renamed /xtal1
- net Net-(C7-Pad2) renamed /xtal2
- net Net-(C8-Pad1) renamed /UCAP
- net Net-(R1-Pad2) renamed /RESET
- net Net-(R4-Pad2) renamed /D2+
- net Net-(R5-Pad2) renamed /D2-
- net Net-(R6-Pad1) renamed /HWB/PE2
- J1 pad A4: VCC -> Net-(J1-PadA4)
- J1 pad B4: VCC -> Net-(J1-PadA4)
Routing:
- net VCC: track 0.00 -> 129.8 mm, vias 0 -> 3
- net /D2-: track 0.00 -> 58.3 mm, vias 0 -> 1
- net /D2+: track 0.00 -> 55.8 mm, vias 0 -> 1
- net col1: track 0.00 -> 40.6 mm
- net row2: track 0.00 -> 38.6 mm
- net row1: track 0.00 -> 38.6 mm
- net D-: track 0.00 -> 19.1 mm
- net D+: track 0.00 -> 19.1 mm
- net col2: track 0.00 -> 19.0 mm
- net col0: track 0.00 -> 19.0 mm
- net Net-(D1-Pad2): track 0.00 -> 12.7 mm
- net /xtal1: track 0.00 -> 8.66 mm
- net /xtal2: track 0.00 -> 8.25 mm
- net /RESET: track 0.00 -> 7.63 mm
- net Net-(J1-PadA4): track 0.00 -> 7.05 mm
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Other:
- board outline added: 68.6 x 76.2 mm

Commit message: save changes
Parts:
- removed C1, C2, C3, C4: 0.1uF, Capacitor_SMD:C_0805_2012Metric_Pad1.18x1.45mm_HandSolder
- removed C5: 10uF, Capacitor_SMD:C_0805_2012Metric_Pad1.18x1.45mm_HandSolder
- removed C6, C7: 22pF, Capacitor_SMD:C_0805_2012Metric_Pad1.18x1.45mm_HandSolder
- removed C8: 1uF, Capacitor_SMD:C_0805_2012Metric_Pad1.18x1.45mm_HandSolder
- removed F1: 500mA, Fuse:Fuse_1206_3216Metric_Pad1.42x1.75mm_HandSolder
- removed MX1, MX2, MX3, MX4, MX5, MX6: MX-NoLED, MX_Only:MXOnly-1U-Hotswap
- removed R1, R6: 10k, Resistor_SMD:R_0805_2012Metric_Pad1.20x1.40mm_HandSolder
- removed R2, R3: 5.1k, Resistor_SMD:R_0805_2012Metric_Pad1.20x1.40mm_HandSolder
- removed R4, R5: 22, Resistor_SMD:R_0805_2012Metric_Pad1.20x1.40mm_HandSolder
- removed Y1: 16MHz, Crystal:Crystal_SMD_SeikoEpson_TSX3225-4Pin_3.2x2.5mm_HandSoldering
- added D10: D_Small, reversible-kicad-footprints:D_SOD-123, F.Cu at (385.5, 191.6)
- added D11: D_Small, reversible-kicad-footprints:D_SOD-123, F.Cu at (468.2, 116.4)
- added D12: D_Small, reversible-kicad-footprints:D_SOD-123, F.Cu at (438.9, 154.6)
- added D13: D_Small, reversible-kicad-footprints:D_SOD-123, F.Cu at (380.9, 211.8)
- added D14: D_Small, reversible-kicad-footprints:D_SOD-123, F.Cu at (512.3, 75.3)
- added D15: D_Small, reversible-kicad-footprints:D_SOD-123, F.Cu at (482.7, 104.2)
- added D16: D_Small, reversible-kicad-footprints:D_SOD-123, F.Cu at (471.9, 122.7)
- added D17: D_Small, reversible-kicad-footprints:D_SOD-123, F.Cu at (475.9, 116.4)
- added D18: D_Small, reversible-kicad-footprints:D_SOD-123, F.Cu at (471.9, 119.5)
- added D19: D_Small, reversible-kicad-footprints:D_SOD-123, F.Cu at (373.2, 215.0)
- added D20: D_Small, reversible-kicad-footprints:D_SOD-123, F.Cu at (400.8, 191.6)
- added D21: D_Small, reversible-kicad-footprints:D_SOD-123, F.Cu at (455.1, 138.0)
- added D22: D_Small, reversible-kicad-footprints:D_SOD-123, F.Cu at (395.0, 197.9)
- added D23: D_Small, reversible-kicad-footprints:D_SOD-123, F.Cu at (387.4, 194.8)
- added D24: D_Small, reversible-kicad-footprints:D_SOD-123, F.Cu at (367.2, 226.2)
- added D25: D_Small, reversible-kicad-footprints:D_SOD-123, F.Cu at (464.2, 124.6)
- added D26: D_Small, reversible-kicad-footprints:D_SOD-123, F.Cu at (407.6, 173.6)
- added D27: D_Small, reversible-kicad-footprints:D_SOD-123, F.Cu at (427.8, 164.8)
- added D28: D_Small, reversible-kicad-footprints:D_SOD-123, F.Cu at (387.4, 204.2)
- added D29: D_Small, reversible-kicad-footprints:D_SOD-123, F.Cu at (479.3, 111.3)
- added D30: D_Small, reversible-kicad-footprints:D_SOD-123, F.Cu at (519.9, 75.3)
- added D31: D_Small, reversible-kicad-footprints:D_SOD-123, F.Cu at (438.9, 148.3)
- added D32: D_Small, reversible-kicad-footprints:D_SOD-123, F.Cu at (459.1, 131.7)
- added D33: D_Small, reversible-kicad-footprints:D_SOD-123, F.Cu at (499.5, 85.5)
- added D34: D_Small, reversible-kicad-footprints:D_SOD-123, F.Cu at (464.2, 121.5)
- added D35: D_Small, reversible-kicad-footprints:D_SOD-123, F.Cu at (407.6, 179.9)
- added D36: D_Small, reversible-kicad-footprints:D_SOD-123, F.Cu at (519.9, 78.4)
- added D37: D_Small, reversible-kicad-footprints:D_SOD-123, F.Cu at (416.8, 168.5)
- added D38: D_Small, reversible-kicad-footprints:D_SOD-123, F.Cu at (374.8, 218.2)
- added D39: D_Small, reversible-kicad-footprints:D_SOD-123, F.Cu at (407.6, 183.0)
- added D40: D_Small, reversible-kicad-footprints:D_SOD-123, F.Cu at (407.6, 186.2)
- added D41: D_Small, reversible-kicad-footprints:D_SOD-123, F.Cu at (459.1, 134.8)
- added D42: D_Small, reversible-kicad-footprints:D_SOD-123, F.Cu at (490.3, 101.1)
- added D43: D_Small, reversible-kicad-footprints:D_SOD-123, F.Cu at (435.4, 158.5)
- added D44: D_Small, reversible-kicad-footprints:D_SOD-123, F.Cu at (424.4, 168.5)
- added D45: D_Small, reversible-kicad-footprints:D_SOD-123, F.Cu at (482.7, 107.4)
- added D46: D_Small, reversible-kicad-footprints:D_SOD-123, F.Cu at (395.0, 194.8)
- added D47: D_Small, reversible-kicad-footprints:D_SOD-123, F.Cu at (499.5, 88.6)
- added D48: D_Small, reversible-kicad-footprints:D_SOD-123, F.Cu at (507.1, 85.5)
- added D49: D_Small, reversible-kicad-footprints:D_SOD-123, F.Cu at (416.8, 171.6)
- added D50: D_Small, reversible-kicad-footprints:D_SOD-123, F.Cu at (367.2, 223.1)
- added D51: D_Small, reversible-kicad-footprints:D_SOD-123, F.Cu at (444.0, 143.2)
- added D52: D_Small, reversible-kicad-footprints:D_SOD-123, F.Cu at (387.4, 197.9)
- added D53: D_Small, reversible-kicad-footprints:D_SOD-123, F.Cu at (427.8, 161.6)
- added D54: D_Small, reversible-kicad-footprints:D_SOD-123, F.Cu at (387.4, 207.4)
- added D55: D_Small, reversible-kicad-footprints:D_SOD-123, F.Cu at (393.1, 191.6)
- added D56: D_Small, reversible-kicad-footprints:D_SOD-123, F.Cu at (373.2, 211.8)
- added D57: D_Small, reversible-kicad-footprints:D_SOD-123, F.Cu at (427.8, 158.5)
- added D58: D_Small, reversible-kicad-footprints:D_SOD-123, F.Cu at (451.7, 143.2)
- added D59: D_Small, reversible-kicad-footprints:D_SOD-123, F.Cu at (415.2, 177.9)
- added D60: D_Small, reversible-kicad-footprints:D_SOD-123, F.Cu at (367.2, 219.9)
- added D61: D_Small, reversible-kicad-footprints:D_SOD-123, F.Cu at (512.3, 78.4)
- added D62: D_Small, reversible-kicad-footprints:D_SOD-123, F.Cu at (464.2, 127.8)
- added D63: D_Small, reversible-kicad-footprints:D_SOD-123, F.Cu at (446.5, 146.3)
- added D64: D_Small, reversible-kicad-footprints:D_SOD-123, F.Cu at (387.4, 201.1)
- added D8: D_Small, reversible-kicad-footprints:D_SOD-123, F.Cu at (482.7, 101.1)
- added D9: D_Small, reversible-kicad-footprints:D_SOD-123, F.Cu at (499.5, 91.8)
- added J2: HDMI_A, Connector_HDMI:HDMI_A_Contact_Technology_HDMI-19APL2_Horizontal, F.Cu at (148.6, 87.6)
- added LED1: SK6812Mini-E, reversible-kicad-footprints:SK6812Mini-E, F.Cu at (-39.4, 7.62)
- added LED10: SK6812Mini-E, reversible-kicad-footprints:SK6812Mini-E, F.Cu at (1.27, -12.7)
- added LED11: SK6812Mini-E, reversible-kicad-footprints:SK6812Mini-E, F.Cu at (21.6, -12.7)
- added LED12: SK6812Mini-E, reversible-kicad-footprints:SK6812Mini-E, F.Cu at (41.9, -12.7)
- added LED13: SK6812Mini-E, reversible-kicad-footprints:SK6812Mini-E, F.Cu at (62.2, -12.7)
- added LED14: SK6812Mini-E, reversible-kicad-footprints:SK6812Mini-E, F.Cu at (82.5, -12.7)
- added LED15: SK6812Mini-E, reversible-kicad-footprints:SK6812Mini-E, F.Cu at (-39.4, 27.9)
- added LED16: SK6812Mini-E, reversible-kicad-footprints:SK6812Mini-E, F.Cu at (-19.1, 27.9)
- added LED17: SK6812Mini-E, reversible-kicad-footprints:SK6812Mini-E, F.Cu at (1.27, 27.9)
- added LED18: SK6812Mini-E, reversible-kicad-footprints:SK6812Mini-E, F.Cu at (21.6, 27.9)
- added LED19: SK6812Mini-E, reversible-kicad-footprints:SK6812Mini-E, F.Cu at (41.9, 27.9)
- added LED2: SK6812Mini-E, reversible-kicad-footprints:SK6812Mini-E, F.Cu at (-19.1, 7.62)
- added LED20: SK6812Mini-E, reversible-kicad-footprints:SK6812Mini-E, F.Cu at (62.2, 27.9)
- added LED21: SK6812Mini-E, reversible-kicad-footprints:SK6812Mini-E, F.Cu at (82.5, 27.9)
- added LED22: SK6812Mini-E, reversible-kicad-footprints:SK6812Mini-E, F.Cu at (429.5, 154.3)
- added LED23: SK6812Mini-E, reversible-kicad-footprints:SK6812Mini-E, F.Cu at (454.9, 127.6)
- added LED24: SK6812Mini-E, reversible-kicad-footprints:SK6812Mini-E, F.Cu at (469.9, 112.3)
- added LED25: SK6812Mini-E, reversible-kicad-footprints:SK6812Mini-E, F.Cu at (462.3, 97.0)
- added LED26: SK6812Mini-E, reversible-kicad-footprints:SK6812Mini-E, F.Cu at (447.8, 116.0)
- added LED27: SK6812Mini-E, reversible-kicad-footprints:SK6812Mini-E, F.Cu at (418.4, 159.2)
- added LED28: SK6812Mini-E, reversible-kicad-footprints:SK6812Mini-E, F.Cu at (257.8, 75.7)
- added LED29: SK6812Mini-E, reversible-kicad-footprints:SK6812Mini-E, F.Cu at (-39.4, 48.3)
- added LED3: SK6812Mini-E, reversible-kicad-footprints:SK6812Mini-E, F.Cu at (1.27, 7.62)
- added LED30: SK6812Mini-E, reversible-kicad-footprints:SK6812Mini-E, F.Cu at (-19.1, 48.3)
- added LED31: SK6812Mini-E, reversible-kicad-footprints:SK6812Mini-E, F.Cu at (1.27, 48.3)
- added LED32: SK6812Mini-E, reversible-kicad-footprints:SK6812Mini-E, F.Cu at (21.6, 48.3)
- added LED33: SK6812Mini-E, reversible-kicad-footprints:SK6812Mini-E, F.Cu at (41.9, 48.3)
- added LED34: SK6812Mini-E, reversible-kicad-footprints:SK6812Mini-E, F.Cu at (62.2, 48.3)
- added LED35: SK6812Mini-E, reversible-kicad-footprints:SK6812Mini-E, F.Cu at (82.5, 48.3)
- added LED36: SK6812Mini-E, reversible-kicad-footprints:SK6812Mini-E, F.Cu at (473.3, 102.1)
- added LED37: SK6812Mini-E, reversible-kicad-footprints:SK6812Mini-E, F.Cu at (491.9, 76.3)
- added LED38: SK6812Mini-E, reversible-kicad-footprints:SK6812Mini-E, F.Cu at (346.8, 222.8)
- added LED39: SK6812Mini-E, reversible-kicad-footprints:SK6812Mini-E, F.Cu at (407.4, 169.4)
- added LED4: SK6812Mini-E, reversible-kicad-footprints:SK6812Mini-E, F.Cu at (21.6, 7.62)
- added LED40: SK6812Mini-E, reversible-kicad-footprints:SK6812Mini-E, F.Cu at (454.9, 122.5)
- added LED41: SK6812Mini-E, reversible-kicad-footprints:SK6812Mini-E, F.Cu at (490.1, 91.6)
- added LED42: SK6812Mini-E, reversible-kicad-footprints:SK6812Mini-E, F.Cu at (378.0, 207.7)
- added LED43: SK6812Mini-E, reversible-kicad-footprints:SK6812Mini-E, F.Cu at (458.9, 112.3)
- added LED44: SK6812Mini-E, reversible-kicad-footprints:SK6812Mini-E, F.Cu at (484.4, 97.0)
- added LED45: SK6812Mini-E, reversible-kicad-footprints:SK6812Mini-E, F.Cu at (357.8, 222.8)
- added LED46: SK6812Mini-E, reversible-kicad-footprints:SK6812Mini-E, F.Cu at (21.6, 68.6)
- added LED47: SK6812Mini-E, reversible-kicad-footprints:SK6812Mini-E, F.Cu at (41.9, 68.6)
- added LED48: SK6812Mini-E, reversible-kicad-footprints:SK6812Mini-E, F.Cu at (62.2, 68.6)
- added LED49: SK6812Mini-E, reversible-kicad-footprints:SK6812Mini-E, F.Cu at (82.5, 68.6)
- added LED5: SK6812Mini-E, reversible-kicad-footprints:SK6812Mini-E, F.Cu at (41.9, 7.62)
- added LED50: SK6812Mini-E, reversible-kicad-footprints:SK6812Mini-E, F.Cu at (378.0, 197.5)
- added LED51: SK6812Mini-E, reversible-kicad-footprints:SK6812Mini-E, F.Cu at (473.3, 107.2)
- added LED52: SK6812Mini-E, reversible-kicad-footprints:SK6812Mini-E, F.Cu at (473.3, 97.0)
- added LED53: SK6812Mini-E, reversible-kicad-footprints:SK6812Mini-E, F.Cu at (346.8, 233.0)
- added LED54: SK6812Mini-E, reversible-kicad-footprints:SK6812Mini-E, F.Cu at (423.6, 144.1)
- added LED55: SK6812Mini-E, reversible-kicad-footprints:SK6812Mini-E, F.Cu at (438.7, 133.9)
- added LED56: SK6812Mini-E, reversible-kicad-footprints:SK6812Mini-E, F.Cu at (423.6, 139.0)
- added LED57: SK6812Mini-E, reversible-kicad-footprints:SK6812Mini-E, F.Cu at (398.2, 182.4)
- added LED58: SK6812Mini-E, reversible-kicad-footprints:SK6812Mini-E, F.Cu at (407.4, 164.3)
- added LED59: SK6812Mini-E, reversible-kicad-footprints:SK6812Mini-E, F.Cu at (447.8, 110.9)
- added LED6: SK6812Mini-E, reversible-kicad-footprints:SK6812Mini-E, F.Cu at (62.2, 7.62)
- added LED60: SK6812Mini-E, reversible-kicad-footprints:SK6812Mini-E, F.Cu at (502.9, 76.3)
- added LED61: SK6812Mini-E, reversible-kicad-footprints:SK6812Mini-E, F.Cu at (458.9, 117.4)
- added LED62: SK6812Mini-E, reversible-kicad-footprints:SK6812Mini-E, F.Cu at (427.6, 133.9)
- added LED63: SK6812Mini-E, reversible-kicad-footprints:SK6812Mini-E, F.Cu at (429.5, 149.2)
- added LED64: SK6812Mini-E, reversible-kicad-footprints:SK6812Mini-E, F.Cu at (387.2, 187.5)
- added LED7: SK6812Mini-E, reversible-kicad-footprints:SK6812Mini-E, F.Cu at (82.5, 7.62)
- added LED8: SK6812Mini-E, reversible-kicad-footprints:SK6812Mini-E, F.Cu at (-39.4, -12.7)
- added LED9: SK6812Mini-E, reversible-kicad-footprints:SK6812Mini-E, F.Cu at (-19.1, -12.7)
- added SW10: SW_Push, reversible-kicad-footprints:MX-1U-Hotswap, F.Cu at (185.4, -17.8)
- added SW11: SW_Push, reversible-kicad-footprints:MX-1U-Hotswap, F.Cu at (205.7, -17.8)
- added SW12: SW_Push, reversible-kicad-footprints:MX-1U-Hotswap, F.Cu at (226.1, -17.8)
- added SW13: SW_Push, reversible-kicad-footprints:MX-1U-Hotswap, F.Cu at (246.4, -17.8)
- added SW14: SW_Push, reversible-kicad-footprints:MX-1U-Hotswap, F.Cu at (266.7, -17.8)
- added SW15: SW_Push, reversible-kicad-footprints:MX-1U-Hotswap, F.Cu at (-39.4, 2.54)
- added SW16: SW_Push, reversible-kicad-footprints:MX-1U-Hotswap, F.Cu at (-19.1, 2.54)
- added SW17: SW_Push, reversible-kicad-footprints:MX-1U-Hotswap, F.Cu at (1.27, 2.54)
- added SW18: SW_Push, reversible-kicad-footprints:MX-1U-Hotswap, F.Cu at (21.6, 2.54)
- added SW19: SW_Push, reversible-kicad-footprints:MX-1U-Hotswap, F.Cu at (41.9, 2.54)
- added SW20: SW_Push, reversible-kicad-footprints:MX-1U-Hotswap, F.Cu at (62.2, 2.54)
- added SW21: SW_Push, reversible-kicad-footprints:MX-1U-Hotswap, F.Cu at (82.5, 2.54)
- added SW22: SW_Push, reversible-kicad-footprints:MX-1U-Hotswap, F.Cu at (144.8, 2.54)
- added SW23: SW_Push, reversible-kicad-footprints:MX-1U-Hotswap, F.Cu at (165.1, 2.54)
- added SW24: SW_Push, reversible-kicad-footprints:MX-1U-Hotswap, F.Cu at (185.4, 2.54)
- added SW25: SW_Push, reversible-kicad-footprints:MX-1U-Hotswap, F.Cu at (205.7, 2.54)
- added SW26: SW_Push, reversible-kicad-footprints:MX-1U-Hotswap, F.Cu at (226.1, 2.54)
- added SW27: SW_Push, reversible-kicad-footprints:MX-1U-Hotswap, F.Cu at (246.4, 2.54)
- added SW28: SW_Push, reversible-kicad-footprints:MX-1U-Hotswap, F.Cu at (266.7, 2.54)
- added SW29: SW_Push, reversible-kicad-footprints:MX-1U-Hotswap, F.Cu at (-39.4, 22.9)
- added SW3: SW_Push, reversible-kicad-footprints:MX-1U-Hotswap, F.Cu at (1.27, -17.8)
- added SW30: SW_Push, reversible-kicad-footprints:MX-1U-Hotswap, F.Cu at (-19.1, 22.9)
- added SW31: SW_Push, reversible-kicad-footprints:MX-1U-Hotswap, F.Cu at (1.27, 22.9)
- added SW32: SW_Push, reversible-kicad-footprints:MX-1U-Hotswap, F.Cu at (21.6, 22.9)
- added SW33: SW_Push, reversible-kicad-footprints:MX-1U-Hotswap, F.Cu at (41.9, 22.9)
- added SW34: SW_Push, reversible-kicad-footprints:MX-1U-Hotswap, F.Cu at (62.2, 22.9)
- added SW35: SW_Push, reversible-kicad-footprints:MX-1U-Hotswap, F.Cu at (82.5, 22.9)
- added SW36: SW_Push, reversible-kicad-footprints:MX-1U-Hotswap, F.Cu at (144.8, 22.9)
- added SW37: SW_Push, reversible-kicad-footprints:MX-1U-Hotswap, F.Cu at (165.1, 22.9)
- added SW38: SW_Push, reversible-kicad-footprints:MX-1U-Hotswap, F.Cu at (185.4, 22.9)
- added SW39: SW_Push, reversible-kicad-footprints:MX-1U-Hotswap, F.Cu at (205.7, 22.9)
- added SW4: SW_Push, reversible-kicad-footprints:MX-1U-Hotswap, F.Cu at (21.6, -17.8)
- added SW40: SW_Push, reversible-kicad-footprints:MX-1U-Hotswap, F.Cu at (226.1, 22.9)
- added SW41: SW_Push, reversible-kicad-footprints:MX-1U-Hotswap, F.Cu at (246.4, 22.9)
- added SW42: SW_Push, reversible-kicad-footprints:MX-1U-Hotswap, F.Cu at (266.7, 22.9)
- added SW43: SW_Push, reversible-kicad-footprints:MX-1U-Hotswap, F.Cu at (-39.4, 43.2)
- added SW44: SW_Push, reversible-kicad-footprints:MX-1U-Hotswap, F.Cu at (-19.1, 43.2)
- added SW45: SW_Push, reversible-kicad-footprints:MX-1U-Hotswap, F.Cu at (1.27, 43.2)
- added SW46: SW_Push, reversible-kicad-footprints:MX-1U-Hotswap, F.Cu at (21.6, 43.2)
- added SW47: SW_Push, reversible-kicad-footprints:MX-1U-Hotswap, F.Cu at (41.9, 43.2)
- added SW48: SW_Push, reversible-kicad-footprints:MX-1U-Hotswap, F.Cu at (62.2, 43.2)
- added SW49: SW_Push, reversible-kicad-footprints:MX-1U-Hotswap, F.Cu at (82.5, 43.2)
- added SW5: SW_Push, reversible-kicad-footprints:MX-1U-Hotswap, F.Cu at (41.9, -17.8)
- added SW50: SW_Push, reversible-kicad-footprints:MX-1U-Hotswap, F.Cu at (144.8, 43.2)
- added SW51: SW_Push, reversible-kicad-footprints:MX-1U-Hotswap, F.Cu at (165.1, 43.2)
- added SW52: SW_Push, reversible-kicad-footprints:MX-1U-Hotswap, F.Cu at (185.4, 43.2)
- added SW53: SW_Push, reversible-kicad-footprints:MX-1U-Hotswap, F.Cu at (205.7, 43.2)
- added SW54: SW_Push, reversible-kicad-footprints:MX-1U-Hotswap, F.Cu at (226.1, 43.2)
- added SW55: SW_Push, reversible-kicad-footprints:MX-1U-Hotswap, F.Cu at (246.4, 43.2)
- added SW56: SW_Push, reversible-kicad-footprints:MX-1U-Hotswap, F.Cu at (266.7, 43.2)
- added SW57: SW_Push, reversible-kicad-footprints:MX-1U-Hotswap, F.Cu at (21.6, 63.5)
- added SW58: SW_Push, reversible-kicad-footprints:MX-1U-Hotswap, F.Cu at (41.9, 63.5)
- added SW59: SW_Push, reversible-kicad-footprints:MX-1U-Hotswap, F.Cu at (62.2, 63.5)
- added SW6: SW_Push, reversible-kicad-footprints:MX-1U-Hotswap, F.Cu at (62.2, -17.8)
- added SW60: SW_Push, reversible-kicad-footprints:MX-1U-Hotswap, F.Cu at (82.5, 63.5)
- added SW61: SW_Push, reversible-kicad-footprints:MX-1U-Hotswap, F.Cu at (144.8, 63.5)
- added SW62: SW_Push, reversible-kicad-footprints:MX-1U-Hotswap, F.Cu at (165.1, 63.5)
- added SW63: SW_Push, reversible-kicad-footprints:MX-1U-Hotswap, F.Cu at (185.4, 63.5)
- added SW64: SW_Push, reversible-kicad-footprints:MX-1U-Hotswap, F.Cu at (205.7, 63.5)
- added SW65: SW_Push, reversible-kicad-footprints:PushButton_4.5mm, F.Cu at (141.0, -73.7)
- added SW7: SW_Push, reversible-kicad-footprints:MX-1U-Hotswap, F.Cu at (82.5, -17.8)
- added SW8: SW_Push, reversible-kicad-footprints:MX-1U-Hotswap, F.Cu at (144.8, -17.8)
- added SW9: SW_Push, reversible-kicad-footprints:MX-1U-Hotswap, F.Cu at (165.1, -17.8)
- J1: value HRO-TYPE-C -> HDMI_A; footprint reversible-kicad-footprints:HRO-TYPE-C-31-M-12-HandSoldering-NoSBU -> Connector_HDMI:HDMI_A_Contact_Technology_HDMI-19APL2_Horizontal; moved to F.Cu
- SW1: footprint reversible-kicad-footprints:PushButton_4.5mm -> reversible-kicad-footprints:MX-1U-Hotswap
- SW2: value RotaryEncoder_Switch -> SW_Push; footprint reversible-kicad-footprints:EC11_Switch -> reversible-kicad-footprints:MX-1U-Hotswap
- U1: value ATmega32U4-A -> ProMicro; footprint Package_QFP:TQFP-44_10x10mm_P0.8mm -> Keebio-Parts:ArduinoProMicro; moved to F.Cu
- moved D4 417.0 mm to (512.3, 81.6), turned to 0 degrees
- moved D1 374.3 mm to (490.3, 104.2), turned to 0 degrees
- moved D2 359.6 mm to (493.7, 95.7), turned to 0 degrees
- moved D3 305.7 mm to (415.2, 174.8), turned to 0 degrees
- moved D5 304.8 mm to (438.9, 151.4), turned to 0 degrees
- moved D6 295.2 mm to (407.6, 176.7), turned to 0 degrees
- moved D7 277.7 mm to (356.1, 232.1), turned to 0 degrees
- moved U1 202.4 mm to (80.0, -104.1), turned to -90 degrees
- moved SW1 194.4 mm to (-39.4, -17.8), turned to 0 degrees
- moved SW2 163.4 mm to (-19.1, -17.8), turned to 0 degrees
- moved J1 17.1 mm to (76.2, 87.6), turned to 90 degrees
Connections:
- D2 pad 1: row1 -> row0
- D3 pad 1: row1 -> row0
- D4 pad 1: row1 -> row0
- D5 pad 1: row2 -> row0
- D6 pad 1: row2 -> row0
- D7 pad 1: row2 -> row0
- SW1 pad 1: GND -> Net-(D1-Pad2)
- SW1 pad 2: /RESET -> col0
- U1 pad 13: /RESET -> unconnected-(U1-Pad13)
- U1 pad 14: VCC -> unconnected-(U1-Pad14)
- U1 pad 15: GND -> unconnected-(U1-Pad15)
- U1 pad 16: /xtal2 -> unconnected-(U1-Pad16)
- U1 pad 17: /xtal1 -> unconnected-(U1-Pad17)
- U1 pad 2: VCC -> unconnected-(U1-Pad2)
- U1 pad 22: unconnected-(U1-Pad22) -> GND
- U1 pad 23: GND -> Net-(SW65-Pad1)
- U1 pad 24: VCC -> unconnected-(U1-Pad24)
- U1 pad 3: /D2- -> GND
- U1 pad 4: /D2+ -> GND
- U1 pad 5: GND -> unconnected-(U1-Pad5)
- U1 pad 6: /UCAP -> unconnected-(U1-Pad6)
- U1 pad 7: VCC -> unconnected-(U1-Pad7)
Routing:
- net VCC: track 129.8 -> 0.00 mm, vias 3 -> 0
- net /D2-: track 58.3 -> 0.00 mm, vias 1 -> 0
- net /D2+: track 55.8 -> 0.00 mm, vias 1 -> 0
- net col1: track 40.6 -> 0.00 mm
- net row2: track 38.6 -> 0.00 mm
- net row1: track 38.6 -> 0.00 mm
- net D-: track 19.1 -> 0.00 mm
- net D+: track 19.1 -> 0.00 mm
- net col2: track 19.0 -> 0.00 mm
- net col0: track 19.0 -> 0.00 mm
- net Net-(D1-Pad2): track 12.7 -> 0.00 mm
- net /xtal1: track 8.66 -> 0.00 mm
- net /xtal2: track 8.25 -> 0.00 mm
- net /RESET: track 7.63 -> 0.00 mm
- net Net-(J1-PadA4): track 7.05 -> 0.00 mm
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Other:
- board size 68.6 x 76.2 mm -> 10.6 x 5.5 mm
