File: _autosave-rubypad.kicad_pcb (KiCad board)
At the start: 2 copper layers, 32 parts, among them J1 HRO-TYPE-C, SW1 SW_Push, SW2 RotaryEncoder_Switch, U1 ATmega32U4-A, Y1 16MHz

Commit message: adding new parts
Parts:
- moved SW1 121.1 mm to (79.2, 20.3), turned to -90 degrees
- moved C6 102.7 mm to (53.8, 29.0), turned to -90 degrees
- moved C7 101.8 mm to (65.5, 29.0), turned to 90 degrees
- moved Y1 95.9 mm to (59.9, 27.9)
- moved R3 92.2 mm to (38.6, 36.6)
- moved C4 84.8 mm to (63.5, 33.5)
- moved C3 83.9 mm to (50.3, 38.6), turned to 180 degrees
- moved C1 72.2 mm to (68.6, 41.1)
- moved C2 69.2 mm to (68.6, 45.2)
- moved R1 67.7 mm to (79.2, 24.9)
- moved C5 65.4 mm to (64.0, 50.3), turned to 180 degrees
- moved R6 20.2 mm to (50.3, 45.7), turned to 180 degrees
- turned U1 to 180 degrees
