File: rubypad.kicad_sch (KiCad schematic)
At the start: 29 parts, among them SW1 SW_Push, SW2 RotaryEncoder_Switch, U1 ATmega32U4-A, Y1 16MHz

Commit message: rev2 is rev1
Parts:
- added J1: HRO-TYPE-C, reversible-kicad-footprints:HRO-TYPE-C-31-M-12-HandSoldering-NoSBU, symbol reversible-kicad-symbols:HRO-TYPE-C-31-M-12-HandSoldering-NoSBU
- added R2, R3: 5.1k, Resistor_SMD:R_0805_2012Metric_Pad1.20x1.40mm_HandSolder, symbol Device:R_Small
- C1, C2, C3, C4, C5, C6, C7, C8: footprint (none) -> Capacitor_SMD:C_0805_2012Metric_Pad1.18x1.45mm_HandSolder
- D1, D2, D3, D4, D5, D6, D7: footprint (none) -> reversible-kicad-footprints:D_SOD-123
- MX1, MX2, MX3, MX4, MX5, MX6: footprint (none) -> MX_Only:MXOnly-1U-Hotswap
- R1, R6: footprint (none) -> Resistor_SMD:R_0805_2012Metric_Pad1.20x1.40mm_HandSolder
- R4: renamed from R3; footprint (none) -> Resistor_SMD:R_0805_2012Metric_Pad1.20x1.40mm_HandSolder
- R5: renamed from R4; footprint (none) -> Resistor_SMD:R_0805_2012Metric_Pad1.20x1.40mm_HandSolder
- SW1: footprint (none) -> reversible-kicad-footprints:PushButton_4.5mm
- SW2: footprint (none) -> reversible-kicad-footprints:EC11_Switch
- Y1: footprint (none) -> Crystal:Crystal_SMD_3225-4Pin_3.2x2.5mm_HandSoldering
Connections:
- net D+: now also J1.A6 (D+), J1.B6 (D+)
- net D-: now also J1.A7 (D-), J1.B7 (D-)
- net GND: now also J1.A1 (GND), J1.B1 (GND), J1.S1 (SHIELD), R2.1, R3.1
- net VCC: now also J1.A4 (VBUS), J1.B4 (VBUS)
- net encA: now reaches SW2.A
- net encB: now reaches SW2.B
- net encC: now reaches SW2.C
- new net: J1.A5 (CC1), R2.2
- new net: J1.B5 (CC2), R3.2
- no-connect marks 29 -> 26

Commit message: adding new parts
Connections:
- net VCC: now also C1.1, C2.1, C3.1, C4.1, C5.1
Changed lines of the file:
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@@
+    (stroke (width 0) (type default) (color 0 0 0 0))
+  )
+  (wire (pts (xy 229.87 21.59) (xy 232.41 21.59))
     (stroke (width 0) (type default) (color 0 0 0 0))
   )
@@
     (in_bom yes) (on_board yes)
     (property "Reference" "R2" (id 0) (at 62.23 33.02 90))
-    (property "Value" "5.1k" (id 1) (at 68.58 33.02 90))
+    (property "Value" "5.1k" (id 1) (at 67.31 33.02 90))
     (property "Footprint" "Resistor_SMD:R_0805_2012Metric_Pad1.20x1.40mm_HandSolder" (id 2) (at 62.23 35.56 0)
       (effects (font (size 1.27 1.27)) hide)
@@
     (in_bom yes) (on_board yes)
     (property "Reference" "R3" (id 0) (at 62.23 40.64 90))
-    (property "Value" "5.1k" (id 1) (at 68.58 40.64 90))
+    (property "Value" "5.1k" (id 1) (at 67.31 40.64 90))
     (property "Footprint" "Resistor_SMD:R_0805_2012Metric_Pad1.20x1.40mm_HandSolder" (id 2) (at 62.23 38.1 0)
       (effects (font (size 1.27 1.27)) hide)
@@
     (pin "2")
   )
+  (symbol (lib_id "power:VCC") (at 229.87 21.59 0) (unit 1)
+    (in_bom yes) (on_board yes) (fields_autoplaced)
+    (property "Reference" "#PWR?" (id 0) (at 229.87 25.4 0)
+      (effects (font (size 1.27 1.27)) hide)
+    )
+    (property "Value" "VCC" (id 1) (at 229.87 17.9855 0))
+    (property "Footprint" "" (id 2) (at 229.87 21.59 0)
+      (effects (font (size 1.27 1.27)) hide)
+    )
+    (property "Datasheet" "" (id 3) (at 229.87 21.59 0)
+      (effects (font (size 1.27 1.27)) hide)
+    )
+    (pin "1")
+  )
   (symbol (lib_id "Device:R_Small") (at 121.92 52.07 90) (unit 1)
     (in_bom yes) (on_board yes) (fields_autoplaced)
@@
       (reference "#PWR013") (unit 1) (value "GND") (footprint "")
     )
+    (path "/db066797-b21c-4c1c-9591-8c7c549f8087"
+      (reference "#PWR?") (unit 1) (value "VCC") (footprint "")
+    )
     (path "/a4dcce92-13b2-431f-a152-59f699af2f2c"

Commit message: update
Connections:
- net col0: now also U1.29 (PB5)
- net col1: now also U1.30 (PB6)
- net col2: now also U1.31 (PC6)
- no-connect marks 26 -> 23
Changed lines of the file:
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@@
   (no_connect (at 160.02 57.15))
   (no_connect (at 160.02 52.07))
-  (no_connect (at 160.02 49.53))
   (no_connect (at 160.02 44.45))
-  (no_connect (at 160.02 41.91))
-  (no_connect (at 160.02 39.37))
   (no_connect (at 160.02 36.83))
   (no_connect (at 160.02 34.29))
@@
     )
   )
+  (global_label "col0" (shape input) (at 160.02 39.37 0) (fields_autoplaced)
+    (effects (font (size 1.27 1.27)) (justify left))
+    (property "Intersheet References" "${INTERSHEET_REFS}" (id 0) (at 166.5455 39.2906 0)
+      (effects (font (size 1.27 1.27)) (justify left) hide)
+    )
+  )
   (global_label "encB" (shape input) (at 36.83 106.68 180) (fields_autoplaced)
     (effects (font (size 1.27 1.27)) (justify right))
@@
     )
   )
+  (global_label "col1" (shape input) (at 160.02 41.91 0) (fields_autoplaced)
+    (effects (font (size 1.27 1.27)) (justify left))
+    (property "Intersheet References" "${INTERSHEET_REFS}" (id 0) (at 166.5455 41.8306 0)
+      (effects (font (size 1.27 1.27)) (justify left) hide)
+    )
+  )
   (global_label "row1" (shape input) (at 31.75 134.62 180) (fields_autoplaced)
     (effects (font (size 1.27 1.27)) (justify right))
@@
     (effects (font (size 1.27 1.27)) (justify left))
     (property "Intersheet References" "${INTERSHEET_REFS}" (id 0) (at 67.4855 49.6094 0)
+      (effects (font (size 1.27 1.27)) (justify left) hide)
+    )
+  )
+  (global_label "col2" (shape input) (at 160.02 49.53 0) (fields_autoplaced)
+    (effects (font (size 1.27 1.27)) (justify left))
+    (property "Intersheet References" "${INTERSHEET_REFS}" (id 0) (at 166.5455 49.4506 0)
       (effects (font (size 1.27 1.27)) (justify left) hide)
     )
@@
   (symbol (lib_id "power:VCC") (at 229.87 21.59 0) (unit 1)
     (in_bom yes) (on_board yes) (fields_autoplaced)
-    (property "Reference" "#PWR?" (id 0) (at 229.87 25.4 0)
+    (property "Reference" "#PWR0101" (id 0) (at 229.87 25.4 0)
       (effects (font (size 1.27 1.27)) hide)
     )
@@
     )
     (path "/db066797-b21c-4c1c-9591-8c7c549f8087"
-      (reference "#PWR?") (unit 1) (value "VCC") (footprint "")
+      (reference "#PWR0101") (unit 1) (value "VCC") (footprint "")
     )
     (path "/a4dcce92-13b2-431f-a152-59f699af2f2c"

Commit message: add to schematic
Other:
- moved on the sheet: C1, C2, C3, C4, C5

Commit message: changes and complete
Connections:
- net col0: now also U1.20 (PD2); no longer U1.29 (PB5)
- net col1: now also U1.21 (PD3); no longer U1.30 (PB6)
- net col2: now also U1.22 (PD5); no longer U1.31 (PC6)
- net encA: now also U1.38 (PF5)
- net encB: now also U1.40 (PF1)
- net encC: now also U1.39 (PF4)
- net row0: now also U1.28 (PB4)
- net row1: now also U1.29 (PB5)
- net row2: now also U1.30 (PB6)
- no-connect marks 23 -> 17
Changed lines of the file:
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@@
   (no_connect (at 160.02 74.93))
   (no_connect (at 160.02 72.39))
-  (no_connect (at 160.02 69.85))
   (no_connect (at 160.02 67.31))
-  (no_connect (at 160.02 64.77))
-  (no_connect (at 160.02 95.25))
-  (no_connect (at 160.02 92.71))
-  (no_connect (at 160.02 90.17))
   (no_connect (at 160.02 87.63))
   (no_connect (at 160.02 82.55))
-  (no_connect (at 160.02 62.23))
   (no_connect (at 160.02 59.69))
   (no_connect (at 160.02 57.15))
   (no_connect (at 160.02 52.07))
   (no_connect (at 160.02 44.45))
-  (no_connect (at 160.02 36.83))
   (no_connect (at 160.02 34.29))
   (no_connect (at 160.02 31.75))
   (no_connect (at 160.02 29.21))
   (no_connect (at 160.02 26.67))
+  (no_connect (at 160.02 49.53))
   (wire (pts (xy 73.66 124.46) (xy 73.66 142.24))
     (stroke (width 0) (type default) (color 0 0 0 0))
@@
     )
   )
-  (global_label "col0" (shape input) (at 160.02 39.37 0) (fields_autoplaced)
-    (effects (font (size 1.27 1.27)) (justify left))
-    (property "Intersheet References" "${INTERSHEET_REFS}" (id 0) (at 166.5455 39.2906 0)
+  (global_label "col1" (shape input) (at 160.02 64.77 0) (fields_autoplaced)
+    (effects (font (size 1.27 1.27)) (justify left))
+    (property "Intersheet References" "${INTERSHEET_REFS}" (id 0) (at 166.5455 64.6906 0)
       (effects (font (size 1.27 1.27)) (justify left) hide)
     )
@@
     )
   )
+  (global_label "col0" (shape input) (at 160.02 62.23 0) (fields_autoplaced)
+    (effects (font (size 1.27 1.27)) (justify left))
+    (property "Intersheet References" "${INTERSHEET_REFS}" (id 0) (at 166.5455 62.1506 0)
+      (effects (font (size 1.27 1.27)) (justify left) hide)
+    )
+  )
   (global_label "col2" (shape input) (at 73.66 91.44 90) (fields_autoplaced)
     (effects (font (size 1.27 1.27)) (justify left))
@@
     )
   )
-  (global_label "col1" (shape input) (at 160.02 41.91 0) (fields_autoplaced)
-    (effects (font (size 1.27 1.27)) (justify left))
-    (property "Intersheet References" "${INTERSHEET_REFS}" (id 0) (at 166.5455 41.8306 0)
+  (global_label "encC" (shape input) (at 160.02 92.71 0) (fields_autoplaced)
+    (effects (font (size 1.27 1.27)) (justify left))
+    (property "Intersheet References" "${INTERSHEET_REFS}" (id 0) (at 167.0293 92.7894 0)
       (effects (font (size 1.27 1.27)) (justify left) hide)
     )
@@
     )
   )
+  (global_label "row2" (shape input) (at 160.02 41.91 0) (fields_autoplaced)
+    (effects (font (size 1.27 1.27)) (justify left))
+    (property "Intersheet References" "${INTERSHEET_REFS}" (id 0) (at 166.9083 41.9894 0)
+      (effects (font (size 1.27 1.27)) (justify left) hide)
+    )
+  )
+  (global_label "encB" (shape input) (at 160.02 90.17 0) (fields_autoplaced)
+    (effects (font (size 1.27 1.27)) (justify left))
+    (property "Intersheet References" "${INTERSHEET_REFS}" (id 0) (at 167.0293 90.2494 0)
+      (effects (font (size 1.27 1.27)) (justify left) hide)
+    )
+  )
+  (global_label "col2" (shape input) (at 160.02 69.85 0) (fields_autoplaced)
+    (effects (font (size 1.27 1.27)) (justify left))
+    (property "Intersheet References" "${INTERSHEET_REFS}" (id 0) (at 166.5455 69.7706 0)
+      (effects (font (size 1.27 1.27)) (justify left) hide)
+    )
+  )
   (global_label "D+" (shape input) (at 62.23 49.53 0) (fields_autoplaced)
     (effects (font (size 1.27 1.27)) (justify left))
@@
     )
   )
-  (global_label "col2" (shape input) (at 160.02 49.53 0) (fields_autoplaced)
-    (effects (font (size 1.27 1.27)) (justify left))
-    (property "Intersheet References" "${INTERSHEET_REFS}" (id 0) (at 166.5455 49.4506 0)
-      (effects (font (size 1.27 1.27)) (justify left) hide)
-    )
-  )
   (global_label "D-" (shape input) (at 107.95 54.61 180) (fields_autoplaced)
     (effects (font (size 1.27 1.27)) (justify right))
@@
     )
   )
+  (global_label "row0" (shape input) (at 160.02 36.83 0) (fields_autoplaced)
+    (effects (font (size 1.27 1.27)) (justify left))
+    (property "Intersheet References" "${INTERSHEET_REFS}" (id 0) (at 166.9083 36.9094 0)
+      (effects (font (size 1.27 1.27)) (justify left) hide)
+    )
+  )
   (global_label "encA" (shape input) (at 36.83 101.6 180) (fields_autoplaced)
     (effects (font (size 1.27 1.27)) (justify right))
@@
     )
   )
+  (global_label "encA" (shape input) (at 160.02 95.25 0) (fields_autoplaced)
+    (effects (font (size 1.27 1.27)) (justify left))
+    (property "Intersheet References" "${INTERSHEET_REFS}" (id 0) (at 166.8479 95.3294 0)
+      (effects (font (size 1.27 1.27)) (justify left) hide)
+    )
+  )
   (global_label "encC" (shape input) (at 36.83 104.14 180) (fields_autoplaced)
     (effects (font (size 1.27 1.27)) (justify right))
@@
     )
   )
+  (global_label "row1" (shape input) (at 160.02 39.37 0) (fields_autoplaced)
+    (effects (font (size 1.27 1.27)) (justify left))
+    (property "Intersheet References" "${INTERSHEET_REFS}" (id 0) (at 166.9083 39.4494 0)
+      (effects (font (size 1.27 1.27)) (justify left) hide)
+    )
+  )

Commit message: udpate - going to redo pcb again
Parts:
- Y1: footprint Crystal:Crystal_SMD_3225-4Pin_3.2x2.5mm_HandSoldering -> Crystal:Crystal_SMD_SeikoEpson_TSX3225-4Pin_3.2x2.5mm_HandSoldering
Changed lines of the file:
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@@
     (property "Reference" "Y1" (id 0) (at 114.3 33.02 90))
     (property "Value" "16MHz" (id 1) (at 114.3 35.56 90))
-    (property "Footprint" "Crystal:Crystal_SMD_3225-4Pin_3.2x2.5mm_HandSoldering" (id 2) (at 106.68 34.29 0)
+    (property "Footprint" "Crystal:Crystal_SMD_SeikoEpson_TSX3225-4Pin_3.2x2.5mm_HandSoldering" (id 2) (at 106.68 34.29 0)
       (effects (font (size 1.27 1.27)) hide)
     )
@@
     )
     (path "/a3f5d478-605e-4e12-a2a8-da8d8a4a13a3"
-      (reference "Y1") (unit 1) (value "16MHz") (footprint "Crystal:Crystal_SMD_3225-4Pin_3.2x2.5mm_HandSoldering")
-    )
-  )
+      (reference "Y1") (unit 1) (value "16MHz") (footprint "Crystal:Crystal_SMD_SeikoEpson_TSX3225-4Pin_3.2x2.5mm_HandSoldering")
+    )
+  )

Commit message: udpate
Connections:
- net col0: no longer U1.20 (PD2)
- net col1: no longer U1.21 (PD3)
- net col2: no longer U1.22 (PD5)
- net encA: no longer U1.38 (PF5)
- net encB: no longer U1.40 (PF1)
- net encC: no longer U1.39 (PF4)
- net row0: no longer U1.28 (PB4)
- net row1: no longer U1.29 (PB5)
- net row2: no longer U1.30 (PB6)
- no-connect marks 17 -> 26
Changed lines of the file:
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@@
   (no_connect (at 160.02 26.67))
   (no_connect (at 160.02 49.53))
+  (no_connect (at 160.02 95.25))
+  (no_connect (at 160.02 92.71))
+  (no_connect (at 160.02 90.17))
+  (no_connect (at 160.02 39.37))
+  (no_connect (at 160.02 41.91))
+  (no_connect (at 160.02 64.77))
+  (no_connect (at 160.02 62.23))
+  (no_connect (at 160.02 69.85))
+  (no_connect (at 160.02 36.83))
   (wire (pts (xy 73.66 124.46) (xy 73.66 142.24))
     (stroke (width 0) (type default) (color 0 0 0 0))
@@
     (property "Intersheet References" "${INTERSHEET_REFS}" (id 0) (at 24.8617 152.3206 0)
       (effects (font (size 1.27 1.27)) (justify right) hide)
-    )
-  )
-  (global_label "col1" (shape input) (at 160.02 64.77 0) (fields_autoplaced)
-    (effects (font (size 1.27 1.27)) (justify left))
-    (property "Intersheet References" "${INTERSHEET_REFS}" (id 0) (at 166.5455 64.6906 0)
-      (effects (font (size 1.27 1.27)) (justify left) hide)
     )
   )
@@
     )
   )
-  (global_label "col0" (shape input) (at 160.02 62.23 0) (fields_autoplaced)
-    (effects (font (size 1.27 1.27)) (justify left))
-    (property "Intersheet References" "${INTERSHEET_REFS}" (id 0) (at 166.5455 62.1506 0)
-      (effects (font (size 1.27 1.27)) (justify left) hide)
-    )
-  )
   (global_label "col2" (shape input) (at 73.66 91.44 90) (fields_autoplaced)
     (effects (font (size 1.27 1.27)) (justify left))
@@
     )
   )
-  (global_label "encC" (shape input) (at 160.02 92.71 0) (fields_autoplaced)
-    (effects (font (size 1.27 1.27)) (justify left))
-    (property "Intersheet References" "${INTERSHEET_REFS}" (id 0) (at 167.0293 92.7894 0)
-      (effects (font (size 1.27 1.27)) (justify left) hide)
-    )
-  )
   (global_label "row1" (shape input) (at 31.75 134.62 180) (fields_autoplaced)
     (effects (font (size 1.27 1.27)) (justify right))
     (property "Intersheet References" "${INTERSHEET_REFS}" (id 0) (at 24.8617 134.5406 0)
       (effects (font (size 1.27 1.27)) (justify right) hide)
-    )
-  )
-  (global_label "row2" (shape input) (at 160.02 41.91 0) (fields_autoplaced)
-    (effects (font (size 1.27 1.27)) (justify left))
-    (property "Intersheet References" "${INTERSHEET_REFS}" (id 0) (at 166.9083 41.9894 0)
-      (effects (font (size 1.27 1.27)) (justify left) hide)
-    )
-  )
-  (global_label "encB" (shape input) (at 160.02 90.17 0) (fields_autoplaced)
-    (effects (font (size 1.27 1.27)) (justify left))
-    (property "Intersheet References" "${INTERSHEET_REFS}" (id 0) (at 167.0293 90.2494 0)
-      (effects (font (size 1.27 1.27)) (justify left) hide)
-    )
-  )
-  (global_label "col2" (shape input) (at 160.02 69.85 0) (fields_autoplaced)
-    (effects (font (size 1.27 1.27)) (justify left))
-    (property "Intersheet References" "${INTERSHEET_REFS}" (id 0) (at 166.5455 69.7706 0)
-      (effects (font (size 1.27 1.27)) (justify left) hide)
     )
   )
@@
     )
   )
-  (global_label "row0" (shape input) (at 160.02 36.83 0) (fields_autoplaced)
-    (effects (font (size 1.27 1.27)) (justify left))
-    (property "Intersheet References" "${INTERSHEET_REFS}" (id 0) (at 166.9083 36.9094 0)
-      (effects (font (size 1.27 1.27)) (justify left) hide)
-    )
-  )
   (global_label "encA" (shape input) (at 36.83 101.6 180) (fields_autoplaced)
     (effects (font (size 1.27 1.27)) (justify right))
@@
     )
   )
-  (global_label "encA" (shape input) (at 160.02 95.25 0) (fields_autoplaced)
-    (effects (font (size 1.27 1.27)) (justify left))
-    (property "Intersheet References" "${INTERSHEET_REFS}" (id 0) (at 166.8479 95.3294 0)
-      (effects (font (size 1.27 1.27)) (justify left) hide)
-    )
-  )
   (global_label "encC" (shape input) (at 36.83 104.14 180) (fields_autoplaced)
     (effects (font (size 1.27 1.27)) (justify right))
@@
     )
   )
-  (global_label "row1" (shape input) (at 160.02 39.37 0) (fields_autoplaced)
-    (effects (font (size 1.27 1.27)) (justify left))
-    (property "Intersheet References" "${INTERSHEET_REFS}" (id 0) (at 166.9083 39.4494 0)
-      (effects (font (size 1.27 1.27)) (justify left) hide)
-    )
-  )
